Commit message: Added prefix to sdh with default to empty prefix for backward compatibility

File: schunk_description/urdf/sdh/sdh.gazebo.xacro (robot description, xacro)
@@ -1,50 +1,51 @@
 <?xml version="1.0"?>
 <robot xmlns:xacro="http://www.ros.org/wiki/xacro">
-  <xacro:macro name="schunk_sdh_gazebo" params="name">
-    <gazebo reference="${name}_palm_link">
+  <xacro:macro name="schunk_sdh_gazebo" params="name prefix:=''">
+    <xacro:property name="prefix_" value="${'' if prefix=='' else prefix+'_'}"/>
+    <gazebo reference="${prefix_}${name}_palm_link">
       <gravity>true</gravity>
       <self_collide>false</self_collide>
       <material>Schunk/LightGrey</material>
     </gazebo>
-    <gazebo reference="${name}_finger_11_link">
+    <gazebo reference="${prefix_}${name}_finger_11_link">
       <gravity>true</gravity>
       <self_collide>false</self_collide>
       <material>Schunk/LightGrey</material>
     </gazebo>
-    <gazebo reference="${name}_finger_12_link">
+    <gazebo reference="${prefix_}${name}_finger_12_link">
       <gravity>true</gravity>
       <self_collide>false</self_collide>
       <material>Schunk/LightGrey</material>
-      <sensor name='${name}_finger_12_contact_sensor' type='contact'>
+      <sensor name='${prefix_}${name}_finger_12_contact_sensor' type='contact'>
         <always_on>true</always_on>
         <update_rate>100</update_rate>
         <contact>
-          <collision>${name}_finger_12_link_collision</collision>
-          <topic>${name}_finger_12_bumper</topic>
+          <collision>${prefix_}${name}_finger_12_link_collision</collision>
+          <topic>${prefix_}${name}_finger_12_bumper</topic>
         </contact>
-        <plugin name="${name}_finger_12_gazebo_ros_bumper_controller" filename="libgazebo_ros_bumper.so">
-          <frameName>${name}_finger_12_link</frameName>
-          <bumperTopicName>${name}_finger_12_bumper</bumperTopicName>
+        <plugin name="${prefix_}${name}_finger_12_gazebo_ros_bumper_controller" filename="libgazebo_ros_bumper.so">
+          <frameName>${prefix_}${name}_finger_12_link</frameName>
+          <bumperTopicName>${prefix_}${name}_finger_12_bumper</bumperTopicName>
         </plugin>
       </sensor>
     </gazebo>
-    <gazebo reference="${name}_finger_13_link">
+    <gazebo reference="${prefix_}${name}_finger_13_link">
       <gravity>true</gravity>
       <self_collide>false</self_collide>
       <material>Schunk/LightGrey</material>
-      <sensor name='${name}_finger_13_contact_sensor' type='contact'>
+      <sensor name='${prefix_}${name}_finger_13_contact_sensor' type='contact'>
         <always_on>true</always_on>
         <update_rate>100</update_rate>
         <contact>
-          <collision>${name}_finger_13_link_collision</collision>
-          <topic>${name}_finger_13_bumper</topic>
+          <collision>${prefix_}${name}_finger_13_link_collision</collision>
+          <topic>${prefix_}${name}_finger_13_bumper</topic>
         </contact>
-        <plugin name="${name}_finger_13_gazebo_ros_bumper_controller" filename="libgazebo_ros_bumper.so">
-          <frameName>${name}_finger_13_link</frameName>
-          <bumperTopicName>${name}_finger_13_bumper</bumperTopicName>
+        <plugin name="${prefix_}${name}_finger_13_gazebo_ros_bumper_controller" filename="libgazebo_ros_bumper.so">
+          <frameName>${prefix_}${name}_finger_13_link</frameName>
+          <bumperTopicName>${prefix_}${name}_finger_13_bumper</bumperTopicName>
         </plugin>
       </sensor>
     </gazebo>
-    <gazebo reference="${name}_finger_21_link">
+    <gazebo reference="${prefix_}${name}_finger_21_link">
       <gravity>true</gravity>
       <self_collide>false</self_collide>
@@ -55,78 +56,78 @@
       <kd value="1.0" /-->
     </gazebo>
-    <gazebo reference="${name}_finger_22_link">
+    <gazebo reference="${prefix_}${name}_finger_22_link">
       <gravity>true</gravity>
       <self_collide>false</self_collide>
       <material>Schunk/LightGrey</material>
-      <sensor name='${name}_finger_22_contact_sensor' type='contact'>
+      <sensor name='${prefix_}${name}_finger_22_contact_sensor' type='contact'>
         <always_on>true</always_on>
         <update_rate>100</update_rate>
         <contact>
-          <collision>${name}_finger_22_link_collision</collision>
-          <topic>${name}_finger_22_bumper</topic>
+          <collision>${prefix_}${name}_finger_22_link_collision</collision>
+          <topic>${prefix_}${name}_finger_22_bumper</topic>
         </contact>
-        <plugin name="${name}_finger_22_gazebo_ros_bumper_controller" filename="libgazebo_ros_bumper.so">
-          <frameName>${name}_finger_22_link</frameName>
-          <bumperTopicName>${name}_finger_22_bumper</bumperTopicName>
+        <plugin name="${prefix_}${name}_finger_22_gazebo_ros_bumper_controller" filename="libgazebo_ros_bumper.so">
+          <frameName>${prefix_}${name}_finger_22_link</frameName>
+          <bumperTopicName>${prefix_}${name}_finger_22_bumper</bumperTopicName>
         </plugin>
       </sensor>
     </gazebo>
-    <gazebo reference="${name}_finger_23_link">
+    <gazebo reference="${prefix_}${name}_finger_23_link">
       <gravity>true</gravity>
       <self_collide>false</self_collide>
       <material>Schunk/LightGrey</material>
-      <sensor name='${name}_finger_23_contact_sensor' type='contact'>
+      <sensor name='${prefix_}${name}_finger_23_contact_sensor' type='contact'>
         <always_on>true</always_on>
         <update_rate>100</update_rate>
         <contact>
-          <collision>${name}_finger_23_link_collision</collision>
-          <topic>${name}_finger_23_bumper</topic>
+          <collision>${prefix_}${name}_finger_23_link_collision</collision>
+          <topic>${prefix_}${name}_finger_23_bumper</topic>
         </contact>
-        <plugin name="${name}_finger_23_gazebo_ros_bumper_controller" filename="libgazebo_ros_bumper.so">
-          <frameName>${name}_finger_23_link</frameName>
-          <bumperTopicName>${name}_finger_23_bumper</bumperTopicName>
+        <plugin name="${prefix_}${name}_finger_23_gazebo_ros_bumper_controller" filename="libgazebo_ros_bumper.so">
+          <frameName>${prefix_}${name}_finger_23_link</frameName>
+          <bumperTopicName>${prefix_}${name}_finger_23_bumper</bumperTopicName>
         </plugin>
       </sensor>
     </gazebo>
-    <gazebo reference="${name}_thumb_1_link">
+    <gazebo reference="${prefix_}${name}_thumb_1_link">
       <gravity>true</gravity>
       <self_collide>false</self_collide>
       <material>Schunk/LightGrey</material>
     </gazebo>
-    <gazebo reference="${name}_thumb_2_link">
+    <gazebo reference="${prefix_}${name}_thumb_2_link">
       <gravity>true</gravity>
       <self_collide>false</self_collide>
       <material>Schunk/LightGrey</material>
-      <sensor name='${name}_thumb_2_contact_sensor' type='contact'>
+      <sensor name='${prefix_}${name}_thumb_2_contact_sensor' type='contact'>
         <always_on>true</always_on>
         <update_rate>100</update_rate>
         <contact>
-          <collision>${name}_thumb_2_link_collision</collision>
-          <topic>${name}_thumb_2_bumper</topic>
+          <collision>${prefix_}${name}_thumb_2_link_collision</collision>
+          <topic>${prefix_}${name}_thumb_2_bumper</topic>
         </contact>
-        <plugin name="${name}_thumb_2_gazebo_ros_bumper_controller" filename="libgazebo_ros_bumper.so">
-          <frameName>${name}_thumb_2_link</frameName>
-          <bumperTopicName>${name}_thumb_2_bumper</bumperTopicName>
+        <plugin name="${prefix_}${name}_thumb_2_gazebo_ros_bumper_controller" filename="libgazebo_ros_bumper.so">
+          <frameName>${prefix_}${name}_thumb_2_link</frameName>
+          <bumperTopicName>${prefix_}${name}_thumb_2_bumper</bumperTopicName>
         </plugin>
       </sensor>
     </gazebo>
-    <gazebo reference="${name}_thumb_3_link">
+    <gazebo reference="${prefix_}${name}_thumb_3_link">
       <gravity>true</gravity>
       <self_collide>false</self_collide>
       <material>Schunk/LightGrey</material>
-      <sensor name='${name}_thumb_3_contact_sensor' type='contact'>
+      <sensor name='${prefix_}${name}_thumb_3_contact_sensor' type='contact'>
         <always_on>true</always_on>
         <update_rate>100</update_rate>
         <contact>
-          <collision>${name}_thumb_3_link_collision</collision>
-          <topic>${name}_thumb_3_bumper</topic>
+          <collision>${prefix_}${name}_thumb_3_link_collision</collision>
+          <topic>${prefix_}${name}_thumb_3_bumper</topic>
         </contact>
-        <plugin name="${name}_thumb_3_gazebo_ros_bumper_controller" filename="libgazebo_ros_bumper.so">
-          <frameName>${name}_thumb_3_link</frameName>
-          <bumperTopicName>${name}_thumb_3_bumper</bumperTopicName>
+        <plugin name="${prefix_}${name}_thumb_3_gazebo_ros_bumper_controller" filename="libgazebo_ros_bumper.so">
+          <frameName>${prefix_}${name}_thumb_3_link</frameName>
+          <bumperTopicName>${prefix_}${name}_thumb_3_bumper</bumperTopicName>
         </plugin>
       </sensor>
     </gazebo>
-    <!--gazebo reference="${name}_finger_21_joint">
+    <!--gazebo reference="${prefix_}${name}_finger_21_joint">
       <stopKd value='1.0' />
       <stopKp value='10000000' />

File: schunk_description/urdf/sdh/sdh.urdf.xacro (robot description, xacro)
@@ -6,12 +6,13 @@
   <!-- will fail to load if already included -->
   <xacro:include filename="$(find schunk_description)/urdf/materials.urdf.xacro" />
-  <xacro:macro name="schunk_sdh" params="parent name *origin">
+  <xacro:macro name="schunk_sdh" params="parent name prefix:='' *origin">
+    <xacro:property name="prefix_" value="${'' if prefix=='' else prefix+'_'}"/>
     <!-- joint between arm_7_link and sdh_palm_link -->
     <joint name="${name}_palm_joint" type="fixed" >
       <xacro:insert_block name="origin" />
       <parent link="${parent}" />
-      <child link="${name}_palm_link" />
-    </joint>
-    <link name="${name}_palm_link">
+      <child link="${prefix_}${name}_palm_link" />
+    </joint>
+    <link name="${prefix_}${name}_palm_link">
       <inertial>
         <mass value="1.0288" /><!-- density 1652.3 kg/m3 adjusted to have final total mass of 1.95 -->
@@ -34,10 +35,10 @@
     </link>
     <!-- grasp link -->
-    <joint name="${name}_grasp_joint" type="fixed" >
+    <joint name="${prefix_}${name}_grasp_joint" type="fixed" >
       <origin xyz="0 0 0.15" rpy="0 0 0"/>
-      <parent link="${name}_palm_link" />
-      <child link="${name}_grasp_link" />
-    </joint>
-    <link name="${name}_grasp_link">
+      <parent link="${prefix_}${name}_palm_link" />
+      <child link="${prefix_}${name}_grasp_link" />
+    </joint>
+    <link name="${prefix_}${name}_grasp_link">
       <xacro:default_inertial/>
       <visual>
@@ -55,10 +56,10 @@
     </link>
     <!-- tip link -->
-    <joint name="${name}_tip_joint" type="fixed" >
+    <joint name="${prefix_}${name}_tip_joint" type="fixed" >
       <origin xyz="0 0 0.22" rpy="0 0 0"/>
-      <parent link="${name}_palm_link" />
-      <child link="${name}_tip_link" />
-    </joint>
-    <link name="${name}_tip_link">
+      <parent link="${prefix_}${name}_palm_link" />
+      <child link="${prefix_}${name}_tip_link" />
+    </joint>
+    <link name="${prefix_}${name}_tip_link">
       <xacro:default_inertial/>
       <visual>
@@ -77,13 +78,13 @@
     <!-- finger1 -->
     <!-- joint between sdh_palm_link and sdh_finger_11_link -->
-    <joint name="${name}_knuckle_joint" type="revolute">
+    <joint name="${prefix_}${name}_knuckle_joint" type="revolute">
       <origin xyz="0.01905 0.033 0.0745" rpy="0 0 3.14159265" />
-      <parent link="${name}_palm_link"/>
-      <child link="${name}_finger_11_link"/>
+      <parent link="${prefix_}${name}_palm_link"/>
+      <child link="${prefix_}${name}_finger_11_link"/>
       <axis xyz="0 0 1" />
       <dynamics damping="1" />
       <limit effort="100" lower="0" upper="1.570796327" velocity="5"/>
     </joint>
-    <link name="${name}_finger_11_link">
+    <link name="${prefix_}${name}_finger_11_link">
       <inertial>
         <mass value="0.047" /> <!-- density of aluminum -->
@@ -106,13 +107,13 @@
     </link>
     <!-- joint between sdh_finger_11_link and sdh_finger_12_link -->
-    <joint name="${name}_finger_12_joint" type="revolute">
+    <joint name="${prefix_}${name}_finger_12_joint" type="revolute">
       <origin xyz="0 0 0.0165" rpy="0 0 0" />
-      <parent link="${name}_finger_11_link"/>
-      <child link="${name}_finger_12_link"/>
-      <axis xyz="0 1 0" />
-      <dynamics damping="1" />
-      <limit effort="100" lower="-1.570796327" upper="1.570796327" velocity="5"/>
-    </joint>
-    <link name="${name}_finger_12_link">
+      <parent link="${prefix_}${name}_finger_11_link"/>
+      <child link="${prefix_}${name}_finger_12_link"/>
+      <axis xyz="0 1 0" />
+      <dynamics damping="1" />
+      <limit effort="100" lower="-1.570796327" upper="1.570796327" velocity="5"/>
+    </joint>
+    <link name="${prefix_}${name}_finger_12_link">
       <inertial>
         <mass value="0.167" /> <!-- density of aluminum -->
@@ -135,13 +136,13 @@
     </link>
     <!-- joint between sdh_finger_12_link and sdh_finger_13_link -->
-    <joint name="${name}_finger_13_joint" type="revolute">
+    <joint name="${prefix_}${name}_finger_13_joint" type="revolute">
       <origin xyz="0 0 0.0865" rpy="0 0 0" />
-      <parent link="${name}_finger_12_link"/>
-      <child link="${name}_finger_13_link"/>
-      <axis xyz="0 1 0" />
-      <dynamics damping="1" />
-      <limit effort="100" lower="-1.570796327" upper="1.570796327" velocity="5"/>
-    </joint>
-    <link name="${name}_finger_13_link">
+      <parent link="${prefix_}${name}_finger_12_link"/>
+      <child link="${prefix_}${name}_finger_13_link"/>
+      <axis xyz="0 1 0" />
+      <dynamics damping="1" />
+      <limit effort="100" lower="-1.570796327" upper="1.570796327" velocity="5"/>
+    </joint>
+    <link name="${prefix_}${name}_finger_13_link">
       <inertial>
         <mass value="0.0929" /> <!-- density of aluminum -->
@@ -165,14 +166,14 @@
     <!-- finger2 -->
     <!-- joint between sdh_palm_link and sdh_finger_21_link -->
-    <joint name="${name}_finger_21_joint" type="revolute">
-      <mimic joint="${name}_knuckle_joint" multiplier="1" offset="0"/>
+    <joint name="${prefix_}${name}_finger_21_joint" type="revolute">
+      <mimic joint="${prefix_}${name}_knuckle_joint" multiplier="1" offset="0"/>
       <origin xyz="0.01905 -0.033 0.0745" rpy="0 0 3.14159265" />
-      <parent link="${name}_palm_link"/>
-      <child link="${name}_finger_21_link"/>
+      <parent link="${prefix_}${name}_palm_link"/>
+      <child link="${prefix_}${name}_finger_21_link"/>
       <axis xyz="0 0 -1" />
       <dynamics damping="1" />
       <limit effort="100" lower="0" upper="1.570796327" velocity="5"/>
     </joint>
-    <link name="${name}_finger_21_link">
+    <link name="${prefix_}${name}_finger_21_link">
       <inertial>
         <mass value="0.047" /> <!-- density of aluminum -->
@@ -195,13 +196,13 @@
     </link>
     <!-- joint between sdh_finger_21_link and sdh_finger_22_link -->
-    <joint name="${name}_finger_22_joint" type="revolute">
+    <joint name="${prefix_}${name}_finger_22_joint" type="revolute">
       <origin xyz="0 0 0.0165" rpy="0 0 0" />
-      <parent link="${name}_finger_21_link"/>
-      <child link="${name}_finger_22_link"/>
-      <axis xyz="0 1 0" />
-      <dynamics damping="1" />
-      <limit effort="100" lower="-1.570796327" upper="1.570796327" velocity="5"/>
-    </joint>
-    <link name="${name}_finger_22_link">
+      <parent link="${prefix_}${name}_finger_21_link"/>
+      <child link="${prefix_}${name}_finger_22_link"/>
+      <axis xyz="0 1 0" />
+      <dynamics damping="1" />
+      <limit effort="100" lower="-1.570796327" upper="1.570796327" velocity="5"/>
+    </joint>
+    <link name="${prefix_}${name}_finger_22_link">
       <inertial>
         <mass value="0.167" /> <!-- density of aluminum -->
@@ -224,13 +225,13 @@
     </link>
     <!-- joint between sdh_finger_22_link and sdh_finger_23_link -->
-    <joint name="${name}_finger_23_joint" type="revolute">
+    <joint name="${prefix_}${name}_finger_23_joint" type="revolute">
       <origin xyz="0 0 0.0865" rpy="0 0 0" />
-      <parent link="${name}_finger_22_link"/>
-      <child link="${name}_finger_23_link"/>
-      <axis xyz="0 1 0" />
-      <dynamics damping="1" />
-      <limit effort="100" lower="-1.570796327" upper="1.570796327" velocity="5"/>
-    </joint>
-    <link name="${name}_finger_23_link">
+      <parent link="${prefix_}${name}_finger_22_link"/>
+      <child link="${prefix_}${name}_finger_23_link"/>
+      <axis xyz="0 1 0" />
+      <dynamics damping="1" />
+      <limit effort="100" lower="-1.570796327" upper="1.570796327" velocity="5"/>
+    </joint>
+    <link name="${prefix_}${name}_finger_23_link">
       <inertial>
         <mass value="0.0929" /> <!-- density of aluminum -->
@@ -254,10 +255,10 @@
     <!-- thumb -->
     <!-- joint between sdh_palm_link and sdh_thumb_1_link -->
-    <joint name="${name}_thumb_1_joint" type="fixed">
+    <joint name="${prefix_}${name}_thumb_1_joint" type="fixed">
       <origin xyz="-0.03811 0 0.0745 " rpy="0 0 0" />
-      <parent link="${name}_palm_link"/>
-      <child link="${name}_thumb_1_link"/>
-    </joint>
-    <link name="${name}_thumb_1_link">
+      <parent link="${prefix_}${name}_palm_link"/>
+      <child link="${prefix_}${name}_thumb_1_link"/>
+    </joint>
+    <link name="${prefix_}${name}_thumb_1_link">
       <inertial>
         <mass value="0.047" /> <!-- density of aluminum -->
@@ -280,13 +281,13 @@
     </link>
     <!-- joint between sdh_thumb_1_link and shd_thumb_2_link -->
-    <joint name="${name}_thumb_2_joint" type="revolute">
+    <joint name="${prefix_}${name}_thumb_2_joint" type="revolute">
     <origin xyz="0 0 0.0165" rpy="0 0 0" />
-    <parent link="${name}_thumb_1_link"/>
-    <child link="${name}_thumb_2_link"/>
+    <parent link="${prefix_}${name}_thumb_1_link"/>
+    <child link="${prefix_}${name}_thumb_2_link"/>
     <axis xyz="0 1 0" />
     <dynamics damping="1" />
     <limit effort="100" lower="-1.570796327" upper="1.570796327" velocity="5"/>
     </joint>
-    <link name="${name}_thumb_2_link">
+    <link name="${prefix_}${name}_thumb_2_link">
       <inertial>
         <mass value="0.167" /> <!-- density of aluminum -->
@@ -309,13 +310,13 @@
     </link>
     <!-- joint between sdh_thumb_2_link and sdh_thumb_3_link -->
-    <joint name="${name}_thumb_3_joint" type="revolute">
+    <joint name="${prefix_}${name}_thumb_3_joint" type="revolute">
       <origin xyz="0 0 0.0865" rpy="0 0 0" />
-      <parent link="${name}_thumb_2_link"/>
-      <child link="${name}_thumb_3_link"/>
-      <axis xyz="0 1 0" />
-      <dynamics damping="1" />
-      <limit effort="100" lower="-1.570796327" upper="1.570796327" velocity="5"/>
-    </joint>
-    <link name="${name}_thumb_3_link">
+      <parent link="${prefix_}${name}_thumb_2_link"/>
+      <child link="${prefix_}${name}_thumb_3_link"/>
+      <axis xyz="0 1 0" />
+      <dynamics damping="1" />
+      <limit effort="100" lower="-1.570796327" upper="1.570796327" velocity="5"/>
+    </joint>
+    <link name="${prefix_}${name}_thumb_3_link">
       <inertial>
         <mass value="0.0929" /> <!-- density of aluminum -->
@@ -338,6 +339,6 @@
     </link>
     <!-- extensions -->
-    <xacro:schunk_sdh_gazebo name="${name}" />
-    <xacro:schunk_sdh_transmission name="${name}" />
+    <xacro:schunk_sdh_gazebo name="${name}" prefix="${prefix}" />
+    <xacro:schunk_sdh_transmission name="${prefix_}${name}" />
   </xacro:macro>
 </robot>
