Commit message: Added reduced collision meshes for knuckles and palm, with no interpenetration

File: schunk_description/urdf/sdh/sdh.urdf.xacro (robot description, xacro)
@@ -23,5 +23,5 @@
         <origin xyz="0 0 0" rpy="0 0 0" />
         <geometry>
-          <mesh filename="package://schunk_description/meshes/sdh/palm.stl"/>
+          <mesh filename="package://schunk_description/meshes/sdh/palm_collision.stl"/>
         </geometry>
       </collision>
@@ -91,5 +91,5 @@
         <origin xyz="0 0 0" rpy="0 0 0" />
         <geometry>
-        <mesh filename="package://schunk_description/meshes/sdh/knuckle.stl"/>
+        <mesh filename="package://schunk_description/meshes/sdh/knuckle_collision.stl"/>
         </geometry>
       </collision>
@@ -168,5 +168,5 @@
         <origin xyz="0 0 0" rpy="0 0 0" />
         <geometry>
-          <mesh filename="package://schunk_description/meshes/sdh/knuckle.stl"/>
+          <mesh filename="package://schunk_description/meshes/sdh/knuckle_collision.stl"/>
         </geometry>
       </collision>
@@ -241,5 +241,5 @@
         <origin xyz="0 0 0" rpy="0 0 0" />
         <geometry>
-          <mesh filename="package://schunk_description/meshes/sdh/knuckle.stl"/>
+          <mesh filename="package://schunk_description/meshes/sdh/knuckle_collision.stl"/>
         </geometry>
       </collision>

Commit message: Added better inertia estimation for sdh (meshlab + aluminum density + adjusted to total mass)

File: schunk_description/urdf/sdh/sdh.urdf.xacro (robot description, xacro)
@@ -12,5 +12,9 @@
     </joint>
     <link name="${name}_palm_link">
-      <xacro:default_inertial/>
+      <inertial>
+        <mass value="1.0288" /><!-- density 1652.3 kg/m3 adjusted to have final total mass of 1.95 -->
+        <origin xyz="0 0 0.0386" />
+        <inertia ixx="0.0011896" ixy="0.0" ixz="0.0" iyy="0.0011889" iyz="0.0" izz="0.0015636" />
+      </inertial>
       <visual>
         <origin xyz="0 0 0" rpy="0 0 0" />
@@ -80,5 +84,9 @@
     </joint>
     <link name="${name}_finger_11_link">
-      <xacro:default_inertial/>
+      <inertial>
+        <mass value="0.047" /> <!-- density of aluminum -->
+        <origin xyz="0.0 2.2105e-03 1.2155e-02" />
+        <inertia ixx="1.5889e-05" ixy="0.0" ixz="0.0" iyy="6.9350e-06" iyz="-4.7500e-07" izz="1.4915e-05" />
+      </inertial>
       <visual>
         <origin xyz="0 0 0" rpy="0 0 0" />
@@ -105,5 +113,9 @@
     </joint>
     <link name="${name}_finger_12_link">
-      <xacro:default_inertial/>
+      <inertial>
+        <mass value="0.167" /> <!-- density of aluminum -->
+        <origin xyz="0.0007467 -0.0000378 0.0430192" />
+        <inertia ixx="1.5920e-04" ixy="0.0" ixz="-2.3750e-08" iyy="1.5903e-04" iyz="9.3100e-06" izz="1.9142e-05" />
+      </inertial>
       <visual>
         <origin xyz="0 0 0" rpy="0 0 0" />
@@ -130,5 +142,9 @@
     </joint>
     <link name="${name}_finger_13_link">
-      <xacro:default_inertial/>
+      <inertial>
+        <mass value="0.0929" /> <!-- density of aluminum -->
+        <origin xyz="0.0007467 -0.0000378 0.0430192" />
+        <inertia ixx="4.2323e-05" ixy="1.9000e-07" ixz="-5.2250e-07" iyy="3.9734e-05" iyz="5.7950e-06" izz="1.1210e-05" />
+      </inertial>
       <visual>
         <origin xyz="0 0 0" rpy="0 0 0" />
@@ -157,5 +173,9 @@
     </joint>
     <link name="${name}_finger_21_link">
-      <xacro:default_inertial/>
+      <inertial>
+        <mass value="0.047" /> <!-- density of aluminum -->
+        <origin xyz="0.0 2.2105e-03 1.2155e-02" />
+        <inertia ixx="1.5889e-05" ixy="0.0" ixz="0.0" iyy="6.9350e-06" iyz="-4.7500e-07" izz="1.4915e-05" />
+      </inertial>
       <visual>
         <origin xyz="0 0 0" rpy="0 0 0" />
@@ -182,5 +202,9 @@
     </joint>
     <link name="${name}_finger_22_link">
-      <xacro:default_inertial/>
+      <inertial>
+        <mass value="0.167" /> <!-- density of aluminum -->
+        <origin xyz="0.0007467 -0.0000378 0.0430192" />
+        <inertia ixx="1.5920e-04" ixy="0.0" ixz="-2.3750e-08" iyy="1.5903e-04" iyz="9.3100e-06" izz="1.9142e-05" />
+      </inertial>
       <visual>
         <origin xyz="0 0 0" rpy="0 0 0" />
@@ -207,5 +231,9 @@
     </joint>
     <link name="${name}_finger_23_link">
-      <xacro:default_inertial/>
+      <inertial>
+        <mass value="0.0929" /> <!-- density of aluminum -->
+        <origin xyz="0.0007467 -0.0000378 0.0430192" />
+        <inertia ixx="4.2323e-05" ixy="1.9000e-07" ixz="-5.2250e-07" iyy="3.9734e-05" iyz="5.7950e-06" izz="1.1210e-05" />
+      </inertial>
       <visual>
         <origin xyz="0 0 0" rpy="0 0 0" />
@@ -230,5 +258,9 @@
     </joint>
     <link name="${name}_thumb_1_link">
-      <xacro:default_inertial/>
+      <inertial>
+        <mass value="0.047" /> <!-- density of aluminum -->
+        <origin xyz="0.0 2.2105e-03 1.2155e-02" />
+        <inertia ixx="1.5889e-05" ixy="0.0" ixz="0.0" iyy="6.9350e-06" iyz="-4.7500e-07" izz="1.4915e-05" />
+      </inertial>
       <visual>
         <origin xyz="0 0 0" rpy="0 0 0" />
@@ -255,5 +287,9 @@
     </joint>
     <link name="${name}_thumb_2_link">
-      <xacro:default_inertial/>
+      <inertial>
+        <mass value="0.167" /> <!-- density of aluminum -->
+        <origin xyz="0.0007467 -0.0000378 0.0430192" />
+        <inertia ixx="1.5920e-04" ixy="0.0" ixz="-2.3750e-08" iyy="1.5903e-04" iyz="9.3100e-06" izz="1.9142e-05" />
+      </inertial>
       <visual>
         <origin xyz="0 0 0" rpy="0 0 0" />
@@ -280,5 +316,9 @@
     </joint>
     <link name="${name}_thumb_3_link">
-      <xacro:default_inertial/>
+      <inertial>
+        <mass value="0.0929" /> <!-- density of aluminum -->
+        <origin xyz="0.0007467 -0.0000378 0.0430192" />
+        <inertia ixx="4.2323e-05" ixy="1.9000e-07" ixz="-5.2250e-07" iyy="3.9734e-05" iyz="5.7950e-06" izz="1.1210e-05" />
+      </inertial>
       <visual>
         <origin xyz="0 0 0" rpy="0 0 0" />
